Commit message: be safe

File: install/my_arm_description/share/my_arm_description/urdf/my_robot.urdf.xacro (robot description, xacro)
@@ -1,5 +1,5 @@
 <?xml version="1.0"?>
 <robot name="my_robot" xmlns:xacro="http://www.ros.org/wiki/xacro">
-     <link name = "base_footprint">
-     </link>
+<xacro:include filename="common.xacro" />
+<xacro:include filename="arm.xacro" />
 </robot>
