Commit message: more safety

File: install/my_arm_description/share/my_arm_description/urdf/arm.xacro (robot description, xacro)
@@ -12,4 +12,22 @@
         </visual>
     </link>
+    <link name="forearm_link">
+            <visual>
+                <geometry>
+                    <cylinder radius="${cylinder_radius}" length="${cylinder_length}"/>
+                </geometry>
+                <origin xyz="0 0 ${(cylinder_length/2)}" rpy="0 0 0"/>
+                <material name="yellow"/>
+            </visual>
+    </link>
+    <link name="hand_link">
+            <visual>
+                <geometry>
+                    <cylinder radius="${cylinder_radius}" length="${cylinder_length}"/>
+                </geometry>
+                <origin xyz="0 0 ${cylinder_length/2}" rpy="0 0 0"/>
+                <material name="orange"/>
+            </visual>
+    </link>
     <joint name="base_joint" type="fixed">
         <parent link="base_footprint"/>
@@ -17,3 +35,17 @@
         <origin xyz="0 0 0" rpy="0 0 0"/>
     </joint>
+    <joint name="base_forearm_joint" type="revolute">
+        <parent link="base_link"/>
+        <child link="forearm_link"/>
+        <origin xyz="0 0 ${(base_height/2)}" rpy="0 0 0"/>
+        <axis xyz="0 1 0"/>
+        <limit effort="1000.0" lower="0" upper="${pi}" velocity="100"/>
+    </joint>
+    <joint name="forearm_hand_joint" type="revolute">
+        <parent link="forearm_link"/>
+        <child link="hand_link"/>
+        <origin xyz="0 0 ${cylinder_length}" rpy="0 0 0"/>
+        <axis xyz="0 1 0"/>
+        <limit effort="1000.0" lower="0" upper="${pi}" velocity="100"/>
+    </joint>
 </robot>

File: install/my_arm_description/share/my_arm_description/urdf/common.xacro (robot description, xacro)
@@ -4,6 +4,6 @@
 <xacro:property name="base_width" value="0.1"/>
 <xacro:property name="base_height" value="0.02"/>
-<xacro:property name="cylinder_radius" value="0.1"/>
-<xacro:property name="cylinder_length" value="0.05"/>
+<xacro:property name="cylinder_radius" value="0.02"/>
+<xacro:property name="cylinder_length" value="0.3"/>
     <material name="white">
         <color rgba="1 1 1 1" />
@@ -20,4 +20,7 @@
     <material name="red">
         <color rgba="1 0 0 1"/>
+    </material>
+    <material name="yellow">
+        <color rgba="1 1 0 1"/>
     </material>
     <xacro:macro name="box_inertia" params="m l w h xyz rpy">

Commit message: more safety

File: install/my_arm_description/share/my_arm_description/urdf/arm.xacro (robot description, xacro)
@@ -11,4 +11,12 @@
             <material name="orange" />
         </visual>
+        <collision>
+            <geometry>
+                <box size="${base_length} ${base_width} ${base_height}"/>
+            </geometry>
+            <origin xyz = "0 0 0" rpy = "0 0 0"/>
+        </collision>
+        <xacro:box_inertia m="0.5" l="${base_length}" w="${base_width}" h="${base_height}"
+                            xyz="0 0 0" rpy="0 0 0"/>
     </link>
     <link name="forearm_link">
@@ -20,4 +28,12 @@
                 <material name="yellow"/>
             </visual>
+            <collision>
+                    <geometry>
+                        <cylinder radius="${cylinder_radius}" length="${cylinder_length}"/>
+                    </geometry>
+                    <origin xyz="0 0 ${(cylinder_length/2)}" rpy="0 0 0"/>
+            </collision>
+        <xacro:wheel_inertia m="0.3" r="${cylinder_radius}" h="${cylinder_length}"
+                             xyz="0 0 ${(cylinder_length/2)}" rpy="0 0 0" />
     </link>
     <link name="hand_link">
@@ -29,4 +45,12 @@
                 <material name="orange"/>
             </visual>
+            <collision>
+                <geometry>
+                    <cylinder radius="${cylinder_radius}" length="${cylinder_length}"/>
+                </geometry>
+                <origin xyz="0 0 ${cylinder_length/2}" rpy="0 0 0"/>
+            </collision>
+        <xacro:wheel_inertia m="0.3" r="${cylinder_radius}" h="${cylinder_length}"
+                             xyz="0 0 ${(cylinder_length/2)}" rpy="0 0 0" />
     </link>
     <joint name="base_joint" type="fixed">
